Commit message: Updated mesh file path

File: cg_ws/src/cg_visualization/urdf/600220.urdf (robot description, URDF)
Before this commit: robot 600220, 1 links, 0 joints
Links:
- link base_link: geometry collision mesh filename=package://cg_visualization/meshes/base_link.STL; visual mesh filename=package://cg_visualization/meshes/base_link.STL

Commit message: Testing changes Apr 17

File: cg_ws/src/cg_visualization/urdf/600220.urdf (robot description, URDF)
Before this commit: robot 600220, 1 links, 0 joints
Links:
- link base_link: geometry collision mesh filename=file:///root/CRATER_GRADER/cg_ws/src/cg_visualization/meshe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; visual mesh filename=file:///root/CRATER_GRADER/cg_ws/src/cg_visualization/meshe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

Commit message: slip seems to work

File: cg_ws/src/cg_visualization/urdf/600220.urdf (robot description, URDF)
Before this commit: robot 600220, 1 links, 0 joints
Links:
- link base_link: geometry visual mesh filename=file:///root/CRATER_GRADER/cg_ws/src/cg_visualization/meshe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 scale=0.001 0.001 0.001
